Commit message: feat: add offline XT16 FAST-LIO profile

File: humble_ws/src/go2w_description/urdf/go2w_description.urdf (robot description, URDF)
Before this commit: robot go2w_description, 36 links, 35 joints
Links:
- added link hesai_lidar
Joints:
- added joint hesai_lidar_joint: type fixed, parent base_link, child hesai_lidar, origin xyz=0.1634 0 0.116 rpy=0 0 1.5707963267948966
